File: pcb/BSPD.kicad_pcb (KiCad board)
At the start: 4 copper layers, 45 x 63.7 mm, 69 parts, among them J1 Test header, J2 T4142012121-000, Q1 AO3400A, SW1 SW_DIP_x03, U1 LM339, U2 LM339, U3 74HC32, U4 74HC02, U5 L7805, U6 L7805

Commit message: Initial Schematic and PCB changes for BR2025
Parts:
- removed C11, C7, C8: 1uF, Capacitor_SMD:C_0402_1005Metric
- removed D4: Blue, LED_SMD:LED_0603_1608Metric
- removed R1, R16, R22: 1k, Resistor_SMD:R_0402_1005Metric
- removed R17, R18: 100k, Resistor_SMD:R_0402_1005Metric
- removed SW1: SW_DIP_x03, Button_Switch_SMD:SW_DIP_SPSTx03_Slide_KingTek_DSHP03TS_W7.62mm_P1.27mm
- added RV9: 10k, Potentiometer_SMD:Potentiometer_Bourns_TC33X_Vertical, F.Cu at (151.5, 95.7)
- added U8: 74HC1G04GV,125, libraries:SOT23-5_FAS, F.Cu at (120.1, 137.0)
- U4: value 74HC02 -> LM339
- moved RV5 2.95 mm to (141.3, 95.7)
- moved RV1 2.95 mm to (118.4, 95.7)
- moved RV2 2.95 mm to (123.5, 95.7)
- moved RV3 2.95 mm to (128.6, 95.7)
- moved RV4 2.95 mm to (136.2, 95.7)
- moved RV6 2.95 mm to (146.3, 95.7)
- moved C6 0.38 mm to (120.1, 118.3)
- moved U4 0.05 mm to (120.1, 113.0), turned to 0 degrees
Connections:
- C6 pad 1: +5V -> Vin
- D3 pad 2: Post-Delay -> FAULT_5V
- J1 pad 3: Startup timer -> unconnected-(J1-Pin_3-Pad3)
- J1 pad 5: Startup button -> unconnected-(J1-Pin_5-Pad5)
- J1 pad 7: /Startup post-delay -> unconnected-(J1-Pin_7-Pad7)
- J2 pad 4: Net-(J2-Pad4) -> GND
- U2 pad 10: VALUE_DELAY -> TPS_in
- U2 pad 11: /Value Pre-Delay -> TPS_THRESH_NEGATIVE
- U2 pad 13: /Value Post-Delay -> Value Error
- U2 pad 14: /Sensor Post-Delay -> (no net)
- U2 pad 8: SENSOR_DELAY -> (no net)
- U2 pad 9: /Sensor Pre-Delay -> (no net)
- U4 pad 1: FAULT_LATCHING -> (no net)
- U4 pad 10: /Startup post-delay -> SENSOR_DELAY
- U4 pad 11: (no net) -> /Sensor Pre-Delay
- U4 pad 12: (no net) -> GND
- U4 pad 13: (no net) -> /Sensor Post-Delay
- U4 pad 14: +5V -> /Value Post-Delay
- U4 pad 2: Post-Delay -> (no net)
- U4 pad 3: Net-(C11-Pad2) -> Vin
- U4 pad 4: FAULT_INV -> (no net)
- U4 pad 5: FAULT_LATCHING -> (no net)
- U4 pad 6: /Startup post-delay -> (no net)
- U4 pad 7: GND -> (no net)
- U4 pad 8: Startup button -> VALUE_DELAY
- U4 pad 9: Startup timer -> /Value Pre-Delay
Routing:
- net TPS_THRESH_NEGATIVE: track 0.00 -> 47.7 mm, vias 0 -> 2
- net Net-(J2-Pad4): track 44.2 -> 0.00 mm, vias 2 -> 0
- net Startup: track 38.2 -> 0.00 mm
- net Startup timer: track 36.7 -> 0.00 mm, vias 1 -> 0
- net /Startup post-delay: track 30.8 -> 0.00 mm, vias 1 -> 0
- net FAULT_LATCHING: track 30.0 -> 0.00 mm, vias 2 -> 0
- net FAULT_INV: track 29.7 -> 0.00 mm, vias 2 -> 0
- net Startup button: track 29.0 -> 0.00 mm
- net Post-Delay: track 95.2 -> 83.3 mm
- net SENSOR_DELAY: track 44.6 -> 49.7 mm
- net +5V: track 54.9 -> 51.0 mm, vias 24 -> 22
- net Net-(C11-Pad2): track 3.82 -> 0.00 mm
- net BSE_THRESH: track 34.0 -> 30.8 mm
- net BSE_HIGH: track 44.3 -> 47.3 mm
- net TPS_LOW: track 38.9 -> 35.9 mm
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Other:
- board text added: "Bronco Racing BSPD Rev. 7"
- board text added: "Noah Banasky Mohammed Afnan November 2024"
- board text removed: "Bronco Racing BSPD Rev. 6"
- board text removed: "Jack LeFevre Jan 2023"
- board text removed: "No Fault"
- board text removed: "No latch"
- board text removed: "Startup"
