File: pcb/power.kicad_sch (KiCad schematic)
At the start: 9 parts, among them U5 L7805, U6 L7805

Commit message: CI/CD Changes
Parts:
- C12, C15, C17, C18: Spice_Model 10u -> (none); Spice_Netlist_Enabled N -> (none); Spice_Primitive C -> (none)
- C14, C16: Spice_Model 0.1u -> (none); Spice_Netlist_Enabled N -> (none); Spice_Primitive C -> (none)

Commit message: Design checklist changes
Parts:
- added D4: SMAJ15CA, Diode_SMD:D_SMA, symbol Diode:SMAJ15CA
Connections:
- net GND: now also D4.1 (A1)
- net Vin: now also D4.2 (A2)
Other:
- note added: "Overvoltage Protection"
